File: faceplates/Amiga Drawbridge BA1/Amiga Drawbridge BA1.kicad_pcb (KiCad board)
At the start: 2 copper layers, 90 x 94 mm, 6 parts, among them M1 Mounting, M2 Mounting, M3 Mounting, M4 Mounting

Commit message: Changed made by notice
Other:
- board text added: "DESIGNED IN LOFOTEN"
- board text removed: "MADE IN LOFOTEN"
