File: faceplates/Greaseweazle FA1/Greaseweazle FA1.kicad_pcb (KiCad board)
At the start: 2 copper layers, 90 x 94 mm, 6 parts, among them M1 Mounting, M2 Mounting, M3 Mounting, M4 Mounting

Commit message: Silkscreen tweaks
Parts:
- moved REF** 1.15 mm to (152.6, 80.2)
Other:
- board text added: "Amiga DrawBridge (Greaseweazle) github.com/tebl"
- board text removed: "Amiga DrawBridge (GreaseWeazle) github.com/tebl"
